File: PCB/Potentiometers/Potentiometers.kicad_sch (KiCad schematic)
At the start: 0 parts

Commit message: PCB Designs
Parts:
- added H1, H2, H3, H4: MountingHole_Pad, MountingHole:MountingHole_3.2mm_M3_DIN965_Pad, symbol Mechanical:MountingHole_Pad
- added J1: Conn_01x05, Connector_PinSocket_2.54mm:PinSocket_1x05_P2.54mm_Vertical, symbol Connector_Generic:Conn_01x05
- added VR1, VR2, VR3: PDB12-H4201-103BF, Control_Panel_Footprints:PDB12H4201103BF, symbol Control_Panel_Symbols:PDB12-H4201-103BF
Connections:
- new net: J1.4 (Pin_4), VR2.2 (WIPER)
- new net: J1.3 (Pin_3), VR3.2 (WIPER)
- new net: J1.5 (Pin_5), VR1.2 (WIPER)
- new net +3.3V: J1.2 (Pin_2), VR1.3 (CW), VR2.3 (CW), VR3.3 (CW)
- new net GND: H1.1, H2.1, H3.1, H4.1, J1.1 (Pin_1), VR1.1 (CCW), VR1.MH1, VR1.MH2, VR2.1 (CCW), VR2.MH1, VR2.MH2, VR3.1 (CCW), VR3.MH1, VR3.MH2
