File: PCB/Switches/Switches.kicad_sch (KiCad schematic)
At the start: 8 parts, among them SW1 SW_SPDT, SW2 SW_SPDT, SW3 SW_SPDT, SW4 SW_SPDT, SW5 SW_SPDT, SW6 SW_SPDT, SW7 SW_SPDT, SW8 SW_SPDT

Commit message: PCB Designs
Parts:
- added H1, H2, H3, H4, H5, H6: MountingHole, MountingHole:MountingHole_3.2mm_M3, symbol Mechanical:MountingHole
- added J1: Conn_01x15, Connector_PinHeader_2.54mm:PinHeader_1x15_P2.54mm_Vertical, symbol Connector_Generic:Conn_01x15
- SW1, SW2, SW3, SW4, SW5, SW6, SW7, SW8: footprint (none) -> Control_Panel_Footprints:100SP4T8B13VS2REH
Connections:
- net at SW4.1 (A): now also J1.6 (Pin_6)
- net +3.3V: now reaches SW4.2 (B)
- net +3.3V: now also SW1.2 (B), SW2.2 (B), SW3.2 (B), SW5.2 (B), SW6.2 (B), SW7.2 (B), SW8.2 (B), J1.1 (Pin_1)
- net at SW4.3 (C): now also J1.7 (Pin_7)
- net at SW1.3 (C): now also J1.2 (Pin_2)
- net at SW2.3 (C): now also J1.3 (Pin_3)
- net at SW6.1 (A): now also J1.10 (Pin_10)
- net at SW6.3 (C): now also J1.11 (Pin_11)
- net at SW8.1 (A): now also J1.14 (Pin_14)
- net at SW8.3 (C): now also J1.15 (Pin_15)
- net at SW3.1 (A): now also J1.4 (Pin_4)
- net at SW3.3 (C): now also J1.5 (Pin_5)
- net at SW5.1 (A): now also J1.8 (Pin_8)
- net at SW5.3 (C): now also J1.9 (Pin_9)
- net at SW7.1 (A): now also J1.12 (Pin_12)
- net at SW7.3 (C): now also J1.13 (Pin_13)
Other:
- moved on the sheet: SW1, SW2, SW3, SW4, SW5, SW6, SW7, SW8
