File: PCB/Switches/Switches.kicad_pcb (KiCad board)
At the start: 2 copper layers, 163 x 95 mm, 15 parts, among them J1 Conn_01x15, SW1 SW_SPDT, SW2 SW_SPDT, SW3 SW_SPDT, SW4 SW_SPDT, SW5 SW_SPDT, SW6 SW_SPDT, SW7 SW_SPDT, SW8 SW_SPDT

Commit message: PCB Manufacturing Files and Full CAD
Other:
- board text added: "Switch Panel: E-SWITCH 100 Series Tolga Cavusoglu September 2025"
Changed lines of the file:
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@@
 		(layer "Edge.Cuts")
+	)
+	(gr_text "Switch Panel: E-SWITCH 100 Series\nTolga Cavusoglu\nSeptember 2025"
+		(at 63.5 57 0)
+		(layer "F.SilkS")
+		(effects
+			(font
+				(size 1 1)
+				(thickness 0.1)
+			)
+			(justify left bottom)
+		)
 	)
 	(segment
