File: PCB/Encoders/Encoders.kicad_pcb (KiCad board)
At the start: 2 copper layers, 80 x 30 mm, 7 parts, among them J1 Conn_01x06, U1 PEC12R-4125F-N0012, U2 PEC12R-4125F-N0012

Commit message: PCB Manufacturing Files and Full CAD
Parts:
- J1: value Conn_01x06 -> Conn_01x05; footprint Connector_PinHeader_2.54mm:PinHeader_1x06_P2.54mm_Vertical -> Connector_PinHeader_2.54mm:PinHeader_1x05_P2.54mm_Vertical
Connections:
- J1 pad 1: GND -> Net-(J1-Pin_1)
- J1 pad 3: Net-(J1-Pin_3) -> GND
- U1 pad A1: Net-(J1-Pin_6) -> Net-(J1-Pin_5)
- U1 pad B1: Net-(J1-Pin_5) -> Net-(J1-Pin_4)
- U1 pad C1: Net-(J1-Pin_4) -> GND
- U2 pad A1: Net-(J1-Pin_3) -> Net-(J1-Pin_2)
- U2 pad B1: Net-(J1-Pin_2) -> Net-(J1-Pin_1)
- U2 pad C1: Net-(J1-Pin_4) -> GND
Routing:
- net Net-(J1-Pin_3): track 27.3 -> 0.00 mm
- net Net-(J1-Pin_1): track 0.00 -> 22.8 mm
- net Net-(J1-Pin_4): track 44.2 -> 24.6 mm
- net Net-(J1-Pin_6): track 17.5 -> 0.00 mm
- net GND: track 131.7 -> 147.1 mm
- net Net-(J1-Pin_2): track 21.7 -> 28.2 mm
- net Net-(J1-Pin_5): track 23.6 -> 18.6 mm
Other:
- board text added: "Encoder Panel: PEC12R-4125F-N0012 Tolga Cavusoglu September 2025"
