File: PCB/Encoders/Encoders.kicad_sch (KiCad schematic)
At the start: 0 parts

Commit message: PCB Designs
Parts:
- added H1, H2, H3, H4: MountingHole_Pad, MountingHole:MountingHole_3.2mm_M3_DIN965_Pad, symbol Mechanical:MountingHole_Pad
- added J1: Conn_01x05, symbol Connector_Generic:Conn_01x05
- added U1, U2: PEC12R-4125F-N0012, Control_Panel_Footprints:PEC12R4125FN0012, symbol Control_Panel_Symbols:PEC12R-4125F-N0012
Connections:
- new net: J1.5 (Pin_5), U1.A1 (CHANNEL_A)
- new net: J1.4 (Pin_4), U1.B1 (CHANNEL_B)
- new net: J1.1 (Pin_1), U2.B1 (CHANNEL_B)
- new net: J1.2 (Pin_2), U2.A1 (CHANNEL_A)
- new net GND: H1.1, H2.1, H3.1, H4.1, J1.3 (Pin_3), U1.1 (MH1), U1.2 (MH2), U1.C1 (COMMON), U2.1 (MH1), U2.2 (MH2), U2.C1 (COMMON)

Commit message: PCB Manufacturing Files and Full CAD
Parts:
- J1: footprint (none) -> Connector_PinHeader_2.54mm:PinHeader_1x05_P2.54mm_Vertical
Changed lines of the file:
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@@
 			)
 		)
-		(property "Footprint" ""
+		(property "Footprint" "Connector_PinHeader_2.54mm:PinHeader_1x05_P2.54mm_Vertical"
 			(at 66.04 77.47 0)
 			(effects
