File: PCB/Buttons/Buttons.kicad_sch (KiCad schematic)
At the start: 0 parts

Commit message: PCB Designs
Parts:
- added C1, C2, C3, C4, C5, C6: 1uf, Capacitor_SMD:C_1206_3216Metric_Pad1.33x1.80mm_HandSolder, symbol Device:C_Small
- added H1, H2, H3, H4: MountingHole, MountingHole:MountingHole_3.2mm_M3, symbol Mechanical:MountingHole
- added J1: Conn_02x11_Odd_Even, Connector_PinSocket_2.54mm:PinSocket_2x11_P2.54mm_Vertical, symbol Connector_Generic:Conn_02x11_Odd_Even
- added S1, S2, S3, S4, S5, S6: ULP12OAP1RSSCL1REDGRN, Control_Panel_Footprints:ULP12OAP1RSSCL1REDGRN, symbol Control_Panel_Symbols:ULP12OAP1RSSCL1REDGRN
Connections:
- new net +3.3V: J1.20 (Pin_20), S1.1 (COM), S2.1 (COM), S3.1 (COM), S4.1 (COM), S5.1 (COM), S6.1 (COM)
- new net +5V: C1.1, C2.1, C3.1, C4.1, C5.1, C6.2, J1.19 (Pin_19), S1.LC1 (COM_A), S2.LC1 (COM_A), S3.LC1 (COM_A), S4.LC1 (COM_A), S5.LC1 (COM_A), S6.LC1 (COM_A)
- new net Buttons0: J1.1 (Pin_1), S1.2 (_N.O.)
- new net Buttons1: J1.3 (Pin_3), S3.2 (_N.O.)
- new net Buttons2: J1.5 (Pin_5), S2.2 (_N.O.)
- new net Buttons3: J1.7 (Pin_7), S4.2 (_N.O.)
- new net Buttons4: J1.9 (Pin_9), S5.2 (_N.O.)
- new net Buttons5: J1.11 (Pin_11), S6.2 (_N.O.)
- new net GND: C1.2, C2.2, C3.2, C4.2, C5.2, C6.1, J1.21 (Pin_21), J1.22 (Pin_22)
- new net LED0: J1.13 (Pin_13), S1.L1 (K_RED)
- new net LED1: J1.15 (Pin_15), S1.L2 (K_GREEN)
- new net LED10: J1.16 (Pin_16), S6.L1 (K_RED)
- new net LED11: J1.18 (Pin_18), S6.L2 (K_GREEN)
- new net LED2: J1.17 (Pin_17), S3.L1 (K_RED)
- new net LED3: J1.2 (Pin_2), S3.L2 (K_GREEN)
- new net LED4: J1.4 (Pin_4), S2.L1 (K_RED)
- new net LED5: J1.6 (Pin_6), S2.L2 (K_GREEN)
- new net LED6: J1.8 (Pin_8), S4.L1 (K_RED)
- new net LED7: J1.10 (Pin_10), S4.L2 (K_GREEN)
- new net LED8: J1.12 (Pin_12), S5.L1 (K_RED)
- new net LED9: J1.14 (Pin_14), S5.L2 (K_GREEN)

Commit message: Update main and button pcbs to fix errors with v1.0
Added pull downs to gpio expander and changed header footprint
Parts:
- J1: footprint Connector_PinSocket_2.54mm:PinSocket_2x11_P2.54mm_Vertical -> Connector_PinHeader_2.54mm:PinHeader_2x11_P2.54mm_Vertical
Changed lines of the file:
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@@
 			)
 		)
-		(property "Footprint" "Connector_PinSocket_2.54mm:PinSocket_2x11_P2.54mm_Vertical"
+		(property "Footprint" "Connector_PinHeader_2.54mm:PinHeader_2x11_P2.54mm_Vertical"
 			(at 62.23 92.71 0)
 			(effects
