File: PCB/Main_Panel/Main_Panel.kicad_sch (KiCad schematic)
At the start: 72 parts, among them IC1 TCA6424ARGJR, J1 Conn_02x11_Odd_Even, J2 Conn_02x11_Odd_Even, J3 Conn_01x05, J4 Conn_01x05, J5 Conn_01x15, U1 Pico, U2 TLC5947DAP

Commit message: Add manufacturing files for v1.1
Parts:
- added R38, R39: 10k, Resistor_SMD:R_0805_2012Metric, symbol Device:R_Small
Connections:
- net GND: now also R38.2, R39.2
- net Switch0: now also R38.1
- net Switch1: now also R39.1
Changed lines of the file:
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@@
 	)
 	(junction
+		(at 38.1 101.6)
+		(diameter 0)
+		(color 0 0 0 0)
+	)
+	(junction
 		(at 148.59 43.18)
 		(diameter 0)
@@
 	)
 	(junction
+		(at 33.02 99.06)
+		(diameter 0)
+		(color 0 0 0 0)
+	)
+	(junction
 		(at 91.44 33.02)
 		(diameter 0)
@@
 	)
 	(junction
+		(at 33.02 109.22)
+		(diameter 0)
+		(color 0 0 0 0)
+	)
+	(junction
 		(at 151.13 45.72)
 		(diameter 0)
@@
 	)
 	(junction
+		(at 38.1 109.22)
+		(diameter 0)
+		(color 0 0 0 0)
+	)
+	(junction
 		(at 124.46 67.31)
 		(diameter 0)
@@
 		)
 	)
+	(wire
+		(pts
+			(xy 33.02 109.22) (xy 33.02 110.49)
+		)
+		(stroke
+			(width 0)
+			(type default)
+		)
+	)
 	(bus
 		(pts
@@
 	(wire
 		(pts
-			(xy 25.4 99.06) (xy 43.18 99.06)
+			(xy 25.4 99.06) (xy 33.02 99.06)
 		)
 		(stroke
@@
 	(wire
 		(pts
+			(xy 33.02 109.22) (xy 33.02 107.95)
+		)
+		(stroke
+			(width 0)
+			(type default)
+		)
+	)
+	(wire
+		(pts
 			(xy 163.83 156.21) (xy 168.91 156.21)
 		)
@@
 	(wire
 		(pts
+			(xy 38.1 109.22) (xy 43.18 109.22)
+		)
+		(stroke
+			(width 0)
+			(type default)
+		)
+	)
+	(wire
+		(pts
 			(xy 148.59 64.77) (xy 148.59 68.58)
 		)
@@
 	(wire
 		(pts
-			(xy 25.4 101.6) (xy 43.18 101.6)
+			(xy 25.4 101.6) (xy 38.1 101.6)
 		)
 		(stroke
@@
 	(wire
 		(pts
+			(xy 38.1 106.68) (xy 38.1 109.22)
+		)
+		(stroke
+			(width 0)
+			(type default)
+		)
+	)
+	(wire
+		(pts
 			(xy 215.9 71.12) (xy 233.68 71.12)
 		)
@@
 	(wire
 		(pts
+			(xy 38.1 101.6) (xy 43.18 101.6)
+		)
+		(stroke
+			(width 0)
+			(type default)
+		)
+	)
+	(wire
+		(pts
 			(xy 151.13 45.72) (xy 162.56 45.72)
 		)
@@
 	(wire
 		(pts
+			(xy 33.02 99.06) (xy 33.02 102.87)
+		)
+		(stroke
+			(width 0)
+			(type default)
+		)
+	)
+	(wire
+		(pts
 			(xy 111.76 67.31) (xy 111.76 69.85)
 		)
@@
 		)
 	)
+	(wire
+		(pts
+			(xy 33.02 99.06) (xy 43.18 99.06)
+		)
+		(stroke
+			(width 0)
+			(type default)
+		)
+	)
 	(bus
 		(pts
@@
 	(wire
 		(pts
+			(xy 38.1 109.22) (xy 33.02 109.22)
+		)
+		(stroke
+			(width 0)
+			(type default)
+		)
+	)
+	(wire
+		(pts
 			(xy 261.62 134.62) (xy 250.19 134.62)
 		)
@@
 	(symbol
 		(lib_id "power:GND")
-		(at 43.18 109.22 270)
+		(at 33.02 110.49 0)
 		(unit 1)
 		(exclude_from_sim no)
@@
 		(fields_autoplaced yes)
 		(property "Reference" "#PWR04"
-			(at 36.83 109.22 0)
+			(at 33.02 116.84 0)
 			(effects
 				(font
@@
 		)
 		(property "Value" "GND"
-			(at 39.37 109.2199 90)
+			(at 35.56 111.7599 0)
 			(effects
 				(font
 					(size 1.27 1.27)
 				)
-				(justify right)
+				(justify left)
 			)
 		)
 		(property "Footprint" ""
-			(at 43.18 109.22 0)
+			(at 33.02 110.49 0)
 			(effects
 				(font
@@
 		)
 		(property "Datasheet" ""
-			(at 43.18 109.22 0)
+			(at 33.02 110.49 0)
 			(effects
 				(font
@@
 		)
 		(property "Description" "Power symbol creates a global label with name \"GND\" , ground"
-			(at 43.18 109.22 0)
+			(at 33.02 110.49 0)
 			(effects
 				(font
@@
 	(symbol
 		(lib_id "Device:R_Small")
+		(at 33.02 105.41 0)
+		(unit 1)
+		(exclude_from_sim no)
+		(in_bom yes)
+		(on_board yes)
+		(dnp no)
+		(property "Reference" "R38"
+			(at 36.322 105.41 90)
+			(effects
+				(font
+					(size 1.016 1.016)
+				)
+				(hide yes)
+			)
+		)
+		(property "Value" "10k"
+			(at 34.798 105.156 90)
+			(effects
+				(font
+					(size 1.27 1.27)
+				)
+			)
+		)
+		(property "Footprint" "Resistor_SMD:R_0805_2012Metric"
+			(at 33.02 105.41 0)
+			(effects
+				(font
+					(size 1.27 1.27)
+				)
+				(hide yes)
+			)
+		)
+		(property "Datasheet" "~"
+			(at 33.02 105.41 0)
+			(effects
+				(font
+					(size 1.27 1.27)
+				)
+				(hide yes)
+			)
+		)
+		(property "Description" "Resistor, small symbol"
+			(at 33.02 105.41 0)
+			(effects
+				(font
+					(size 1.27 1.27)
+				)
+				(hide yes)
+			)
+		)
+		(pin "2"
+		)
+		(pin "1"
+		)
+		(instances
+			(project "Main_Panel"
+				(path "/2d982b0e-52da-4895-98f0-64f69e456399"
+					(reference "R38")
+					(unit 1)
+				)
+			)
+		)
+	)
+	(symbol
+		(lib_id "Device:R_Small")
 		(at 250.19 132.08 0)
 		(unit 1)
@@
 					(unit 1)
 				)
+			)
+		)
+	)
+	(symbol
+		(lib_id "Device:R_Small")
+		(at 38.1 104.14 0)
+		(unit 1)
+		(exclude_from_sim no)
+		(in_bom yes)
+		(on_board yes)
+		(dnp no)
+		(property "Reference" "R39"
+			(at 41.402 104.14 90)
+			(effects
+				(font
+					(size 1.016 1.016)
+				)
+				(hide yes)
+			)
+		)
+		(property "Value" "10k"
+			(at 39.878 103.886 90)
+			(effects
+				(font
+					(size 1.27 1.27)
+				)
+			)
+		)
+		(property "Footprint" "Resistor_SMD:R_0805_2012Metric"
+			(at 38.1 104.14 0)
+			(effects
+				(font
+					(size 1.27 1.27)
+				)
+				(hide yes)
+			)
+		)
+		(property "Datasheet" "~"
+			(at 38.1 104.14 0)
+			(effects
+				(font
+					(size 1.27 1.27)
+				)
+				(hide yes)
+			)
+		)
+		(property "Description" "Resistor, small symbol"
+			(at 38.1 104.14 0)
+			(effects
+				(font
+					(size 1.27 1.27)
+				)
+				(hide yes)
+			)
+		)
+		(pin "2"
+		)
+		(pin "1"
+		)
+		(instances
+			(project "Main_Panel"
+				(path "/2d982b0e-52da-4895-98f0-64f69e456399"
+					(reference "R39")
+					(unit 1)
+				)
